File: Black_Body_Temperature_Sensor_PCB/Black_Body_Temperature_Sensor_PCB.kicad_sch (KiCad schematic)
At the start: 0 parts

Commit message: current source simulation, pcb 2->1 switches
Other:
- added sheet V&I_sense (V&I_sense.kicad_sch)
- added sheet micrcontroller (micrcontroller.kicad_sch)
- added sheet nA_current (nA_current.kicad_sch)
- added sheet power_supply (power_supply.kicad_sch)
- added sheet sensor_interface (sensor_interface.kicad_sch)
- added sheet uA_current (uA_current.kicad_sch)

Commit message: temp sensor pcb progress
Other:
- sheet nA_current ports: added "sel"{100na_neg 100na_pos 10na_neg 10na_pos}, nA_I_Source; removed none
- sheet sensor_interface ports: added hbridge_sel[1..4], i_source_sel[1..4], nA_I_Source, uA_I_Source, v_sense{V+ V-}; removed none
- sheet uA_current ports: added "sel_t"{1mA 100uA 10uA 1uA}, "sel_v"{1mA 100uA 10uA 1uA}, uA_I_Source; removed none
Changed lines of the file:
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@@
 	(generator_version "10.0")
 	(paper "A4")
-	(sheet
-		(at 25.4 101.6)
-		(size 50.8 50.8)
+	(wire
+		(pts
+			(xy 114.3 48.26) (xy 128.27 48.26)
+		)
+		(stroke
+			(width 0)
+			(type default)
+		)
+	)
+	(wire
+		(pts
+			(xy 114.3 72.39) (xy 128.27 72.39)
+		)
+		(stroke
+			(width 0)
+			(type default)
+		)
+	)
+	(sheet
+		(at 54.61 100.33)
+		(size 167.64 22.86)
 		(exclude_from_sim no)
 		(in_bom yes)
@@
 		)
 		(property "Sheetname" "micrcontroller"
-			(at 25.4 100.8884 0)
+			(at 54.61 99.6184 0)
 			(show_name no)
 			(do_not_autoplace no)
@@
 		)
 		(property "Sheetfile" "micrcontroller.kicad_sch"
-			(at 25.4 152.9846 0)
+			(at 54.61 123.7746 0)
 			(show_name no)
 			(do_not_autoplace no)
@@
 	)
 	(sheet
-		(at 101.6 101.6)
-		(size 50.8 50.8)
-		(exclude_from_sim no)
-		(in_bom yes)
-		(on_board yes)
-		(dnp no)
-		(fields_autoplaced yes)
+		(at 128.27 38.1)
+		(size 40.64 41.91)
+		(exclude_from_sim no)
+		(in_bom yes)
+		(on_board yes)
+		(dnp no)
 		(stroke
 			(width 0.1524)
@@
 		)
 		(property "Sheetname" "sensor_interface"
-			(at 101.6 100.8884 0)
+			(at 128.27 37.3884 0)
 			(show_name no)
 			(do_not_autoplace no)
@@
 		)
 		(property "Sheetfile" "sensor_interface.kicad_sch"
-			(at 101.6 152.9846 0)
-			(show_name no)
-			(do_not_autoplace no)
-			(effects
-				(font
-					(size 1.27 1.27)
-				)
-				(justify left top)
+			(at 125.73 81.28 0)
+			(show_name no)
+			(do_not_autoplace no)
+			(effects
+				(font
+					(size 1.27 1.27)
+				)
+				(justify left top)
+			)
+		)
+		(pin "v_sense{V+ V-}" input
+			(at 168.91 48.26 0)
+			(effects
+				(font
+					(size 1.27 1.27)
+				)
+				(justify right)
+			)
+		)
+		(pin "uA_I_Source" input
+			(at 128.27 72.39 180)
+			(effects
+				(font
+					(size 1.27 1.27)
+				)
+				(justify left)
+			)
+		)
+		(pin "nA_I_Source" input
+			(at 128.27 48.26 180)
+			(effects
+				(font
+					(size 1.27 1.27)
+				)
+				(justify left)
+			)
+		)
+		(pin "i_source_sel[1..4]" input
+			(at 162.56 80.01 270)
+			(effects
+				(font
+					(size 1.27 1.27)
+				)
+				(justify left)
+			)
+		)
+		(pin "hbridge_sel[1..4]" input
+			(at 158.75 80.01 270)
+			(effects
+				(font
+					(size 1.27 1.27)
+				)
+				(justify left)
 			)
 		)
@@
 	)
 	(sheet
-		(at 179.07 25.4)
-		(size 49.53 50.8)
+		(at 180.34 38.1)
+		(size 41.91 41.91)
 		(exclude_from_sim no)
 		(in_bom yes)
@@
 		)
 		(property "Sheetname" "V&I_sense"
-			(at 179.07 24.6884 0)
+			(at 180.34 37.3884 0)
 			(show_name no)
 			(do_not_autoplace no)
@@
 		)
 		(property "Sheetfile" "V&I_sense.kicad_sch"
-			(at 179.07 76.7846 0)
+			(at 180.34 80.5946 0)
 			(show_name no)
 			(do_not_autoplace no)
@@
 	)
 	(sheet
-		(at 177.8 101.6)
-		(size 50.8 50.8)
+		(at 242.57 90.17)
+		(size 25.4 24.13)
 		(exclude_from_sim no)
 		(in_bom yes)
@@
 		)
 		(property "Sheetname" "power_supply"
-			(at 177.8 100.8884 0)
+			(at 242.57 89.4584 0)
 			(show_name no)
 			(do_not_autoplace no)
@@
 		)
 		(property "Sheetfile" "power_supply.kicad_sch"
-			(at 177.8 152.9846 0)
+			(at 242.57 114.8846 0)
 			(show_name no)
 			(do_not_autoplace no)
@@
 	)
 	(sheet
-		(at 101.6 25.4)
-		(size 50.8 50.8)
+		(at 54.61 38.1)
+		(size 59.69 16.51)
 		(exclude_from_sim no)
 		(in_bom yes)
@@
 		)
 		(property "Sheetname" "nA_current"
-			(at 101.6 24.6884 0)
+			(at 54.61 37.3884 0)
 			(show_name no)
 			(do_not_autoplace no)
@@
 		)
 		(property "Sheetfile" "nA_current.kicad_sch"
-			(at 101.6 76.7846 0)
-			(show_name no)
-			(do_not_autoplace no)
-			(effects
-				(font
-					(size 1.27 1.27)
-				)
-				(justify left top)
+			(at 54.61 55.1946 0)
+			(show_name no)
+			(do_not_autoplace no)
+			(effects
+				(font
+					(size 1.27 1.27)
+				)
+				(justify left top)
+			)
+		)
+		(pin "nA_I_Source" input
+			(at 114.3 48.26 0)
+			(effects
+				(font
+					(size 1.27 1.27)
+				)
+				(justify right)
+			)
+		)
+		(pin "\"sel\"{100na_neg 100na_pos 10na_neg 10na_pos}" input
+			(at 54.61 44.45 180)
+			(effects
+				(font
+					(size 1.27 1.27)
+				)
+				(justify left)
 			)
 		)
@@
 	)
 	(sheet
-		(at 25.4 25.4)
-		(size 50.8 50.8)
+		(at 54.61 63.5)
+		(size 59.69 16.51)
 		(exclude_from_sim no)
 		(in_bom yes)
@@
 		)
 		(property "Sheetname" "uA_current"
-			(at 25.4 24.6884 0)
+			(at 54.61 62.7884 0)
 			(show_name no)
 			(do_not_autoplace no)
@@
 		)
 		(property "Sheetfile" "uA_current.kicad_sch"
-			(at 25.4 76.7846 0)
-			(show_name no)
-			(do_not_autoplace no)
-			(effects
-				(font
-					(size 1.27 1.27)
-				)
-				(justify left top)
-			)
-		)
+			(at 54.61 80.5946 0)
+			(show_name no)
+			(do_not_autoplace no)
+			(effects
+				(font
+					(size 1.27 1.27)
+				)
+				(justify left top)
+			)
+		)
+		(pin "uA_I_Source" input
+			(at 114.3 72.39 0)
+			(effects
+				(font
+					(size 1.27 1.27)
+				)
+				(justify right)
+			)
+		)
+		(pin "\"sel_v\"{1mA 100uA 10uA 1uA}" input
+			(at 54.61 69.85 180)
+			(effects
+				(font
+					(size 1.27 1.27)
+				)
+				(justify left)
+			)
+		)
+		(pin "\"sel_t\"{1mA 100uA 10uA 1uA}" input
+			(at 54.61 73.66 180)
+			(effects
+				(font
+					(size 1.27 1.27)
+				)
+				(justify left)
+			)
+		)
