File: Black_Body_Temperature_Sensor_PCB/micrcontroller.kicad_sch (KiCad schematic)
At the start: 0 parts

Commit message: temp sensor pcb progress
Parts:
- added C10, C11, C12, C13, C7, C8, C9: 0.1uf, symbol Device:C
- added FB1: FerriteBead, symbol Device:FerriteBead
- added R18, R19: 10k, symbol Device:R
- added SW1, SW2: 430471035826, -switch:430471035826, symbol -switch:SW_Push
- added U4: STM32G431CBTx, Package_QFP:LQFP-48_7x7mm_P0.5mm, symbol MCU_ST_STM32G4:STM32G431CBTx
Connections:
- new net +3V3: C10.1, C11.1, C12.1, C8.1, C9.1, FB1.2, R19.1, U4.1 (VBAT), U4.21 (VDDA), U4.24 (VDD), U4.36 (VDD), U4.48 (VDD)
- new net +3V3A: FB1.1
- new net BOOT0: C13.1, R18.2, SW2.1, U4.45 (PB8)
- new net GNDPWR: C10.2, C11.2, C12.2, C13.2, C7.2, C8.2, C9.2, R18.1, SW1.2, SW2.2, U4.19 (VSSA), U4.23 (VSS), U4.35 (VSS), U4.47 (VSS)
- new net NRST: C7.1, R19.2, SW1.1, U4.7 (PG10)
- new net XTAL0: U4.5 (PF0)
- new net XTAL1: U4.6 (PF1)
- no-connect marks 0 -> 34
