File: Black_Body_Temperature_Sensor_PCB/nA_current.kicad_sch (KiCad schematic)
At the start: 0 parts

Commit message: temp sensor pcb progress
Parts:
- added C1: 200pf, symbol Device:C
- added D1: LT1004-1.2, Package_SO:SOIC-8_3.9x4.9mm_P1.27mm, symbol -diode:LT1004CS8-1.2
- added Q7: TMUX1112PWR, Package_SO:TSSOP-16_4.4x5mm_P0.65mm, symbol -fet:TMUX1112PWR
- added R10: 1M, symbol Device:R
- added R11: 100M, symbol Device:R
- added R12: 10M, symbol Device:R
- added R13: 22.6k, symbol Device:R
- added R14: 100k, symbol Device:R
- added R15: 2.7k, symbol Device:R
- added R9: 226k, symbol Device:R
- added U2: LM334M, Package_SO:SOIC-8_3.9x4.9mm_P1.27mm, symbol Reference_Current:LM334M
- added U3: LT1008, Package_SO:SOIC-8_3.9x4.9mm_P1.27mm, symbol -opamp:LT1008
Connections:
- new net: R10.1, R11.1, R9.2
- new net: R12.1, R13.2, R14.1
- new net: C1.1, U3.8
- new net: R15.1, U2.1
- new net: D1.4, Q7.15 (D2), Q7.2 (D1), U3.2 (-), U3.6
- new net: Q7.12 (NC), Q7.4 (NC)
- new net +3V3: Q7.13 (VDD)
- new net +4V: U2.4, U3.7
- new net -4V: C1.2, U3.4
- new net 100na_neg: Q7.3 (S1), R14.2
- new net 100na_pos: Q7.11 (S3), R12.2
- new net 10na_neg: Q7.14 (S2), R10.2
- new net 10na_pos: Q7.6 (S4), R11.2
- new net GNDPWR: Q7.5 (GND)
- new net V-: D1.6, D1.8, R13.1, R15.2, R9.1, U2.2, U2.3, U2.6, U2.7
- new net nA_I_Source: Q7.10 (D3), Q7.7 (D4), U3.3 (+)
- new net sel.100na_neg: Q7.1 (SEL1)
- new net sel.100na_pos: Q7.9 (SEL3)
- new net sel.10na_neg: Q7.16 (SEL2)
- new net sel.10na_pos: Q7.8 (SEL4)
- no-connect marks 0 -> 1
