File: Black_Body_Temperature_Sensor_PCB/sensor_interface.kicad_sch (KiCad schematic)
At the start: 0 parts

Commit message: temp sensor pcb progress
Parts:
- added J1: Conn_01x04_Pin, symbol Connector:Conn_01x04_Pin
- added Q8, Q9: TMUX1112PWR, Package_SO:TSSOP-16_4.4x5mm_P0.65mm, symbol -fet:TMUX1112PWR
- added R16, R17: 10k, symbol Device:R
Connections:
- new net: Q9.14 (S2), R16.1
- new net: Q9.6 (S4), R17.1
- new net: Q8.11 (S3), Q9.11 (S3)
- new net: Q9.12 (NC), Q9.4 (NC)
- new net: Q8.3 (S1), Q9.3 (S1)
- new net: Q8.12 (NC), Q8.4 (NC)
- new net +3V3: Q8.13 (VDD), Q9.13 (VDD)
- new net GND: Q8.14 (S2), Q8.6 (S4), R16.2, R17.2
- new net GNDPWR: Q8.5 (GND), Q9.5 (GND)
- new net hbridge_sel1: Q8.1 (SEL1)
- new net hbridge_sel2: Q8.16 (SEL2)
- new net hbridge_sel3: Q8.9 (SEL3)
- new net hbridge_sel4: Q8.8 (SEL4)
- new net i+: J1.3 (Pin_3), Q8.15 (D2), Q8.2 (D1)
- new net i-: J1.4 (Pin_4), Q8.10 (D3), Q8.7 (D4)
- new net i_source_sel1: Q9.1 (SEL1)
- new net i_source_sel2: Q9.16 (SEL2)
- new net i_source_sel3: Q9.9 (SEL3)
- new net i_source_sel4: Q9.8 (SEL4)
- new net nA_I_Source: Q9.10 (D3), Q9.7 (D4)
- new net uA_I_Source: Q9.15 (D2), Q9.2 (D1)
- new net v_sense.V+: J1.1 (Pin_1)
- new net v_sense.V-: J1.2 (Pin_2)
