File: Black_Body_Temperature_Sensor_PCB/uA_current.kicad_sch (KiCad schematic)
At the start: 15 parts, among them Q1 TMUX1219-Q1, Q2 TMUX1219-Q1, Q3 TMUX1219-Q1, Q4 TMUX1219-Q1, Q5 TMUX1112PWR, U1 LM334M

Commit message: temp sensor pcb progress
Parts:
- removed Q1, Q2, Q3, Q4: TMUX1219-Q1, Package_TO_SOT_SMD:SOT-23-6, symbol -fet:TMUX1219-Q1
- added Q6: TMUX1112PWR, Package_SO:TSSOP-16_4.4x5mm_P0.65mm, symbol -fet:TMUX1112PWR
Connections:
- net +3V3: now also Q5.13 (VDD), Q6.13 (VDD)
- net 100uA_T: now also Q6.15 (D2)
- net 100uA_V: now also Q5.15 (D2)
- net 10uA_T: now also Q6.10 (D3)
- net 10uA_V: now also Q5.10 (D3)
- net 1mA_T: now also Q6.2 (D1)
- net 1mA_V: now also Q5.2 (D1)
- net 1uA_T: now also Q6.7 (D4)
- net 1uA_V: now also Q5.7 (D4)
- net GNDPWR: now also Q5.5 (GND), Q6.5 (GND)
- net LM334M_V-: now also Q5.11 (S3), Q5.14 (S2), Q5.3 (S1), Q5.6 (S4)
- net sel_v.1mA: now reaches Q5.1 (SEL1)
- net sel_v.100uA: now reaches Q5.16 (SEL2)
- net sel_v.1uA: now reaches Q5.8 (SEL4)
- net sel_v.10uA: now reaches Q5.9 (SEL3)
- net uA_I_source renamed uA_I_Source
- net uA_I_Source: now also Q6.11 (S3), Q6.14 (S2), Q6.3 (S1), Q6.6 (S4)
- new net: Q6.12 (NC), Q6.4 (NC)
- new net sel_t.100uA: Q6.16 (SEL2)
- new net sel_t.10uA: Q6.9 (SEL3)
- new net sel_t.1mA: Q6.1 (SEL1)
- new net sel_t.1uA: Q6.8 (SEL4)
Other:
- moved on the sheet: Q5
