File: Circuit Boards/Black_Body_Temperature_Sensor_PCB/Black_Body_Temperature_Sensor_PCB.kicad_sch (KiCad schematic)
At the start: 0 parts

Commit message: power simulation
Other:
- sheet micrcontroller ports: added "sel"{100na_neg 100na_pos 10na_neg 10na_pos}, "sel_t"{1mA 100uA 10uA 1uA}, "sel_v"{1mA 100uA 10uA 1uA}, hbridge_sel[1..4], i_source_sel[1..4]; removed none
Changed lines of the file:
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@@
 	(generator_version "10.0")
 	(paper "A4")
+	(bus
+		(pts
+			(xy 39.37 111.76) (xy 39.37 69.85)
+		)
+		(stroke
+			(width 0)
+			(type default)
+		)
+	)
+	(bus
+		(pts
+			(xy 162.56 80.01) (xy 162.56 100.33)
+		)
+		(stroke
+			(width 0)
+			(type default)
+		)
+	)
+	(bus
+		(pts
+			(xy 54.61 111.76) (xy 39.37 111.76)
+		)
+		(stroke
+			(width 0)
+			(type default)
+		)
+	)
 	(wire
 		(pts
@@
 		)
 	)
+	(bus
+		(pts
+			(xy 54.61 73.66) (xy 48.26 73.66)
+		)
+		(stroke
+			(width 0)
+			(type default)
+		)
+	)
+	(bus
+		(pts
+			(xy 54.61 44.45) (xy 31.75 44.45)
+		)
+		(stroke
+			(width 0)
+			(type default)
+		)
+	)
 	(wire
 		(pts
 			(xy 114.3 72.39) (xy 128.27 72.39)
+		)
+		(stroke
+			(width 0)
+			(type default)
+		)
+	)
+	(bus
+		(pts
+			(xy 39.37 69.85) (xy 54.61 69.85)
+		)
+		(stroke
+			(width 0)
+			(type default)
+		)
+	)
+	(bus
+		(pts
+			(xy 158.75 80.01) (xy 158.75 100.33)
+		)
+		(stroke
+			(width 0)
+			(type default)
+		)
+	)
+	(bus
+		(pts
+			(xy 31.75 118.11) (xy 54.61 118.11)
+		)
+		(stroke
+			(width 0)
+			(type default)
+		)
+	)
+	(bus
+		(pts
+			(xy 48.26 105.41) (xy 54.61 105.41)
+		)
+		(stroke
+			(width 0)
+			(type default)
+		)
+	)
+	(bus
+		(pts
+			(xy 31.75 44.45) (xy 31.75 118.11)
+		)
+		(stroke
+			(width 0)
+			(type default)
+		)
+	)
+	(bus
+		(pts
+			(xy 48.26 73.66) (xy 48.26 105.41)
 		)
 		(stroke
@@
 			)
 		)
+		(pin "\"sel\"{100na_neg 100na_pos 10na_neg 10na_pos}" input
+			(at 54.61 118.11 180)
+			(effects
+				(font
+					(size 1.27 1.27)
+				)
+				(justify left)
+			)
+		)
+		(pin "hbridge_sel[1..4]" input
+			(at 158.75 100.33 90)
+			(effects
+				(font
+					(size 1.27 1.27)
+				)
+				(justify right)
+			)
+		)
+		(pin "i_source_sel[1..4]" input
+			(at 162.56 100.33 90)
+			(effects
+				(font
+					(size 1.27 1.27)
+				)
+				(justify right)
+			)
+		)
+		(pin "\"sel_t\"{1mA 100uA 10uA 1uA}" input
+			(at 54.61 105.41 180)
+			(effects
+				(font
+					(size 1.27 1.27)
+				)
+				(justify left)
+			)
+		)
+		(pin "\"sel_v\"{1mA 100uA 10uA 1uA}" input
+			(at 54.61 111.76 180)
+			(effects
+				(font
+					(size 1.27 1.27)
+				)
+				(justify left)
+			)
+		)
 		(instances
 			(project "Black_Body_Temperature_Sensor_PCB"
@@
 	)
 	(sheet
-		(at 242.57 90.17)
+		(at 241.3 68.58)
 		(size 25.4 24.13)
 		(exclude_from_sim no)
@@
 		)
 		(property "Sheetname" "power_supply"
-			(at 242.57 89.4584 0)
+			(at 241.3 67.8684 0)
 			(show_name no)
 			(do_not_autoplace no)
@@
 		)
 		(property "Sheetfile" "power_supply.kicad_sch"
-			(at 242.57 114.8846 0)
-			(show_name no)
-			(do_not_autoplace no)
+			(at 241.3 93.2946 0)
+			(show_name no)
+			(do_not_autoplace no)

Commit message: Schematic ready for review
Other:
- sheet V&I_sense ports: added i_sense{I+ I-}, v_sense{V+ V-}; removed none
- sheet micrcontroller ports: added i_sense_sel[1..4]; removed none
- sheet sensor_interface ports: added i_sense_sel[1..4], i_sense{I+ I-}; removed none
Changed lines of the file:
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@@
 	(bus
 		(pts
-			(xy 162.56 80.01) (xy 162.56 100.33)
+			(xy 167.64 50.8) (xy 180.34 50.8)
+		)
+		(stroke
+			(width 0)
+			(type default)
+		)
+	)
+	(bus
+		(pts
+			(xy 161.29 80.01) (xy 161.29 100.33)
 		)
 		(stroke
@@
 	(wire
 		(pts
-			(xy 114.3 48.26) (xy 128.27 48.26)
+			(xy 114.3 48.26) (xy 127 48.26)
 		)
 		(stroke
@@
 		)
 	)
+	(bus
+		(pts
+			(xy 167.64 45.72) (xy 180.34 45.72)
+		)
+		(stroke
+			(width 0)
+			(type default)
+		)
+	)
+	(bus
+		(pts
+			(xy 165.1 80.01) (xy 165.1 100.33)
+		)
+		(stroke
+			(width 0)
+			(type default)
+		)
+	)
 	(wire
 		(pts
-			(xy 114.3 72.39) (xy 128.27 72.39)
+			(xy 114.3 72.39) (xy 127 72.39)
 		)
 		(stroke
@@
 	(bus
 		(pts
-			(xy 158.75 80.01) (xy 158.75 100.33)
+			(xy 157.48 80.01) (xy 157.48 100.33)
 		)
 		(stroke
@@
 		)
 		(pin "hbridge_sel[1..4]" input
-			(at 158.75 100.33 90)
+			(at 157.48 100.33 90)
 			(effects
 				(font
@@
 		)
 		(pin "i_source_sel[1..4]" input
-			(at 162.56 100.33 90)
+			(at 161.29 100.33 90)
 			(effects
 				(font
@@
 				)
 				(justify left)
+			)
+		)
+		(pin "i_sense_sel[1..4]" input
+			(at 165.1 100.33 90)
+			(effects
+				(font
+					(size 1.27 1.27)
+				)
+				(justify right)
 			)
 		)
@@
 			(project "Black_Body_Temperature_Sensor_PCB"
 				(path "/e46fba8d-0294-4f4f-927d-8614bb9d51d3"
-					(page "5")
+					(page "7")
 				)
 			)
@@
 	)
 	(sheet
-		(at 128.27 38.1)
+		(at 127 38.1)
 		(size 40.64 41.91)
 		(exclude_from_sim no)
@@
 		)
 		(property "Sheetname" "sensor_interface"
-			(at 128.27 37.3884 0)
+			(at 127 37.3884 0)
 			(show_name no)
 			(do_not_autoplace no)
@@
 		)
 		(property "Sheetfile" "sensor_interface.kicad_sch"
-			(at 125.73 81.28 0)
+			(at 124.46 81.28 0)
 			(show_name no)
 			(do_not_autoplace no)
@@
 		)
 		(pin "v_sense{V+ V-}" input
-			(at 168.91 48.26 0)
+			(at 167.64 45.72 0)
 			(effects
 				(font
@@
 		)
 		(pin "uA_I_Source" input
-			(at 128.27 72.39 180)
+			(at 127 72.39 180)
 			(effects
 				(font
@@
 		)
 		(pin "nA_I_Source" input
-			(at 128.27 48.26 180)
+			(at 127 48.26 180)
 			(effects
 				(font
@@
 		)
 		(pin "i_source_sel[1..4]" input
-			(at 162.56 80.01 270)
+			(at 161.29 80.01 270)
 			(effects
 				(font
@@
 		)
 		(pin "hbridge_sel[1..4]" input
-			(at 158.75 80.01 270)
+			(at 157.48 80.01 270)
+			(effects
+				(font
+					(size 1.27 1.27)
+				)
+				(justify left)
+			)
+		)
+		(pin "i_sense{I+ I-}" input
+			(at 167.64 50.8 0)
+			(effects
+				(font
+					(size 1.27 1.27)
+				)
+				(justify right)
+			)
+		)
+		(pin "i_sense_sel[1..4]" input
+			(at 165.1 80.01 270)
 			(effects
 				(font
@@
 			(project "Black_Body_Temperature_Sensor_PCB"
 				(path "/e46fba8d-0294-4f4f-927d-8614bb9d51d3"
-					(page "6")
+					(page "4")
 				)
 			)
@@
 			)
 		)
+		(pin "v_sense{V+ V-}" input
+			(at 180.34 45.72 180)
+			(effects
+				(font
+					(size 1.27 1.27)
+				)
+				(justify left)
+			)
+		)
+		(pin "i_sense{I+ I-}" input
+			(at 180.34 50.8 180)
+			(effects
+				(font
+					(size 1.27 1.27)
+				)
+				(justify left)
+			)
+		)
 		(instances
 			(project "Black_Body_Temperature_Sensor_PCB"
 				(path "/e46fba8d-0294-4f4f-927d-8614bb9d51d3"
-					(page "4")
+					(page "5")
 				)
 			)
@@
 	)
 	(sheet
-		(at 241.3 68.58)
-		(size 25.4 24.13)
+		(at 231.14 38.1)
+		(size 41.91 41.91)
 		(exclude_from_sim no)
 		(in_bom yes)
@@
 		)
 		(property "Sheetname" "power_supply"
-			(at 241.3 67.8684 0)
+			(at 231.14 37.3884 0)
 			(show_name no)
 			(do_not_autoplace no)
@@
 		)
 		(property "Sheetfile" "power_supply.kicad_sch"
-			(at 241.3 93.2946 0)
+			(at 231.14 80.5946 0)
 			(show_name no)
 			(do_not_autoplace no)
@@
 			(project "Black_Body_Temperature_Sensor_PCB"
 				(path "/e46fba8d-0294-4f4f-927d-8614bb9d51d3"
-					(page "7")
-				)
-			)
+					(page "6")
+				)
+			)

Commit message: Temperature Sensor Schematic Done, awaiting review
Other:
- sheet V&I_sense ports: added ADC_DRDY, CLK_MCO, SPI{SCLK, MOSI, MISO, CS}; removed none
- sheet micrcontroller ports: added ADC_DRDY, CLK_MCO, SPI{SCLK, MOSI, MISO, CS}; removed none
Changed lines of the file:
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@@
 	(generator_version "10.0")
 	(paper "A4")
+	(wire
+		(pts
+			(xy 229.87 72.39) (xy 229.87 107.95)
+		)
+		(stroke
+			(width 0)
+			(type default)
+		)
+	)
 	(bus
 		(pts
@@
 	(bus
 		(pts
+			(xy 226.06 104.14) (xy 222.25 104.14)
+		)
+		(stroke
+			(width 0)
+			(type default)
+		)
+	)
+	(bus
+		(pts
 			(xy 54.61 111.76) (xy 39.37 111.76)
 		)
@@
 		)
 	)
+	(wire
+		(pts
+			(xy 222.25 68.58) (xy 234.95 68.58)
+		)
+		(stroke
+			(width 0)
+			(type default)
+		)
+	)
 	(bus
 		(pts
@@
 	(bus
 		(pts
+			(xy 222.25 76.2) (xy 226.06 76.2)
+		)
+		(stroke
+			(width 0)
+			(type default)
+		)
+	)
+	(wire
+		(pts
+			(xy 222.25 72.39) (xy 229.87 72.39)
+		)
+		(stroke
+			(width 0)
+			(type default)
+		)
+	)
+	(wire
+		(pts
+			(xy 229.87 107.95) (xy 222.25 107.95)
+		)
+		(stroke
+			(width 0)
+			(type default)
+		)
+	)
+	(bus
+		(pts
 			(xy 167.64 45.72) (xy 180.34 45.72)
 		)
@@
 	(bus
 		(pts
+			(xy 226.06 76.2) (xy 226.06 104.14)
+		)
+		(stroke
+			(width 0)
+			(type default)
+		)
+	)
+	(wire
+		(pts
+			(xy 234.95 68.58) (xy 234.95 111.76)
+		)
+		(stroke
+			(width 0)
+			(type default)
+		)
+	)
+	(bus
+		(pts
 			(xy 165.1 80.01) (xy 165.1 100.33)
 		)
@@
 		(pts
 			(xy 114.3 72.39) (xy 127 72.39)
+		)
+		(stroke
+			(width 0)
+			(type default)
+		)
+	)
+	(wire
+		(pts
+			(xy 234.95 111.76) (xy 222.25 111.76)
 		)
 		(stroke
@@
 			)
 		)
+		(pin "SPI{SCLK, MOSI, MISO, CS}" input
+			(at 222.25 104.14 0)
+			(effects
+				(font
+					(size 1.27 1.27)
+				)
+				(justify right)
+			)
+		)
+		(pin "ADC_DRDY" input
+			(at 222.25 107.95 0)
+			(effects
+				(font
+					(size 1.27 1.27)
+				)
+				(justify right)
+			)
+		)
+		(pin "CLK_MCO" input
+			(at 222.25 111.76 0)
+			(effects
+				(font
+					(size 1.27 1.27)
+				)
+				(justify right)
+			)
+		)
 		(instances
 			(project "Black_Body_Temperature_Sensor_PCB"
@@
 			)
 		)
+		(pin "SPI{SCLK, MOSI, MISO, CS}" input
+			(at 222.25 76.2 0)
+			(effects
+				(font
+					(size 1.27 1.27)
+				)
+				(justify right)
+			)
+		)
+		(pin "ADC_DRDY" input
+			(at 222.25 72.39 0)
+			(effects
+				(font
+					(size 1.27 1.27)
+				)
+				(justify right)
+			)
+		)
+		(pin "CLK_MCO" input
+			(at 222.25 68.58 0)
+			(effects
+				(font
+					(size 1.27 1.27)
+				)
+				(justify right)
+			)
+		)
 		(instances
 			(project "Black_Body_Temperature_Sensor_PCB"
@@
 	)
 	(sheet
-		(at 231.14 38.1)
-		(size 41.91 41.91)
+		(at 241.3 38.1)
+		(size 38.1 38.1)
 		(exclude_from_sim no)
 		(in_bom yes)
@@
 		)
 		(property "Sheetname" "power_supply"
-			(at 231.14 37.3884 0)
+			(at 241.3 37.3884 0)
 			(show_name no)
 			(do_not_autoplace no)
@@
 		)
 		(property "Sheetfile" "power_supply.kicad_sch"
-			(at 231.14 80.5946 0)
-			(show_name no)
-			(do_not_autoplace no)
+			(at 241.3 76.7846 0)
+			(show_name no)
+			(do_not_autoplace no)

Commit message: Temp sensor schematic done
Other:
- note added: "OVERVIEW (PAGE 1)"
Changed lines of the file:
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@@
 	(generator_version "10.0")
 	(paper "A4")
+	(text "OVERVIEW (PAGE 1)"
+		(exclude_from_sim no)
+		(at 69.85 24.13 0)
+		(effects
+			(font
+				(size 7 7)
+			)
+		)
+	)
 	(wire
 		(pts
