File: Circuit Boards/Black_Body_Temperature_Sensor_PCB/power_supply.kicad_sch (KiCad schematic)
At the start: 4 parts, among them J3 Barrel_Jack, U5 AMS1117-3.3

Commit message: Schematic ready for review
Parts:
- removed C4, C5: C, symbol Device:C
- removed U5: AMS1117-3.3, Package_TO_SOT_SMD:SOT-223-3_TabPin2, symbol Regulator_Linear:AMS1117-3.3
- added C18, C22, C23, C28, C6: 10uf, symbol Device:C
- added C19: 1uf, symbol Device:C
- added C20, C21: 10nf, symbol Device:C
- added C24, C25, C26, C27: 4.7uf, symbol Device:C
- added D3: D, symbol Device:D
- added R22, R25: 570k, symbol Device:R
- added R23, R24: 180k, symbol Device:R
- added R26, R31: 200k, symbol Device:R
- added R27: 499, symbol Device:R
- added R28, R32: 33.2k, symbol Device:R
- added R29: 453k, symbol Device:R
- added R30: 49.9k, symbol Device:R
- added R33: 7.5k, symbol Device:R
- added R34: 450k, symbol Device:R
- added R35: 50k, symbol Device:R
- added U6: LTC3260xMSE, Package_SO:MSOP-16-1EP_3x4.039mm_P0.5mm_EP1.651x2.845mm, symbol Regulator_SwitchedCapacitor:LTC3260xMSE
- added U7: LT3042xMSE, Package_SO:MSOP-10-1EP_3x3mm_P0.5mm_EP1.68x1.88mm, symbol Regulator_Linear:LT3042xMSE
- added U8: LT3094xMSE, Package_SO:MSOP-12-1EP_3x4.039mm_P0.65mm_EP1.651x2.845mm, symbol Regulator_Linear:LT3094xMSE
Connections:
- net 5Vin renamed 12Vin
- net 12Vin: now also C6.1, D3.1 (K), U6.1 (EN^{+}), U6.11 (V_{IN}), U6.13 (EN^{-})
- net GNDPWR renamed GND
- net GND: now also C18.2, C20.1, C21.2, C22.2, C23.1, C24.2, C25.2, C26.1, C27.2, C28.2, C6.2, D3.2 (A), R23.2, R24.1, R27.1, R28.1, R30.1, R32.1, R33.1, R35.1, U6.14 (MODE), U6.17 (GND), U6.2 (RT), U7.11 (GND), U7.8 (GND), U8.9 (GND)
- new net: C21.1, U6.16 (BYP^{+})
- new net: C18.1, U6.6 (V_{OUT})
- new net: R24.2, R25.1, U6.4 (ADJ^{-})
- new net: R31.1, U8.4 (PG)
- new net: R34.1, R35.2, U8.5 (PGFB)
- new net: R33.2, U8.6 (ILIM)
- new net: C27.1, R32.2, U8.8 (SET)
- new net: R29.1, R30.2, U7.6 (PGFB)
- new net: R26.1, U7.4 (PG)
- new net: R27.2, U7.5 (ILIM)
- new net: C25.1, R28.2, U7.7 (SET)
- new net: R22.2, R23.1, U6.15 (ADJ^{+})
- new net: C19.1, U6.10 (C^{+})
- new net: C20.2, U6.3 (BYP^{-})
- new net: C19.2, U6.7 (C^{-})
- new net +3V3A: C26.2, R29.2, U7.10 (OUT), U7.9 (OUTS)
- new net +5VA: C23.2, C24.1, R22.1, R26.2, R31.2, U6.12 (LDO^{+}), U7.1 (IN), U7.2 (IN), U7.3 (EN/UV)
- new net -3V3A: R34.2, U8.10 (OUTS), U8.11 (OUT), U8.12 (OUT)
- new net -5VA: C22.1, C28.1, R25.2, U6.5 (LDO^{-}), U8.1 (IN), U8.13 (IN), U8.2 (IN), U8.3 (EN/UV)
- no-connect marks 0 -> 1
Other:
- note added: "+12V in -> +5V & -5V 100uV noise"
- note added: "+5V in -> +3V3 0.8uV noise"
- note added: "-5V in -> -3V3 0.8uV noise"
- note removed: "Microcontroller 3.3V"
- moved on the sheet: J3

Commit message: Temp sensor schematic done
Parts:
- removed D3: D, symbol Device:D
- removed J3: Barrel_Jack, symbol Connector:Barrel_Jack
- added P601: 436500200, -connector:436500200 2-pin, symbol -connector:436500200
- C601: renamed from C6; footprint (none) -> Capacitor_SMD:C_0603_1608Metric
- C602: renamed from C18; footprint (none) -> Capacitor_SMD:C_0603_1608Metric
- C603: renamed from C19; footprint (none) -> Capacitor_SMD:C_0603_1608Metric
- C604: renamed from C21; footprint (none) -> Capacitor_SMD:C_0603_1608Metric
- C605: renamed from C20; footprint (none) -> Capacitor_SMD:C_0603_1608Metric
- C606: renamed from C23; footprint (none) -> Capacitor_SMD:C_0603_1608Metric
- C607: renamed from C22; footprint (none) -> Capacitor_SMD:C_0603_1608Metric
- C608: renamed from C24; footprint (none) -> Capacitor_SMD:C_0603_1608Metric
- C609: renamed from C28; footprint (none) -> Capacitor_SMD:C_0603_1608Metric
- C610: renamed from C27; footprint (none) -> Capacitor_SMD:C_0603_1608Metric
- C611: renamed from C25; footprint (none) -> Capacitor_SMD:C_0603_1608Metric
- C612: renamed from C26; footprint (none) -> Capacitor_SMD:C_0603_1608Metric
- R601: renamed from R22; footprint (none) -> Resistor_SMD:R_0603_1608Metric
- R602: renamed from R23; footprint (none) -> Resistor_SMD:R_0603_1608Metric
- R603: renamed from R24; footprint (none) -> Resistor_SMD:R_0603_1608Metric
- R604: renamed from R25; footprint (none) -> Resistor_SMD:R_0603_1608Metric
- R605: renamed from R32; footprint (none) -> Resistor_SMD:R_0603_1608Metric
- R606: renamed from R27; footprint (none) -> Resistor_SMD:R_0603_1608Metric
- R607: renamed from R31; footprint (none) -> Resistor_SMD:R_0603_1608Metric
- R608: renamed from R28; footprint (none) -> Resistor_SMD:R_0603_1608Metric
- R609: renamed from R26; footprint (none) -> Resistor_SMD:R_0603_1608Metric
- R610: renamed from R33; footprint (none) -> Resistor_SMD:R_0603_1608Metric
- R611: renamed from R29; footprint (none) -> Resistor_SMD:R_0603_1608Metric
- R612: renamed from R30; footprint (none) -> Resistor_SMD:R_0603_1608Metric
- R613: renamed from R34; footprint (none) -> Resistor_SMD:R_0603_1608Metric
- R614: renamed from R35; footprint (none) -> Resistor_SMD:R_0603_1608Metric
- renumbered U6 to U601, U8 to U602, U7 to U603
Connections:
- net 12Vin: now also P601.1
- net GND: now also P601.2
Other:
- note added: "Power Supply (PAGE 6)"

Commit message: temp pcb analog layout done
Changed lines of the file:
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@@
+		)
+	)
+	(text_box "Add diode and pi filter"
+		(exclude_from_sim no)
+		(at 57.15 91.44 0)
+		(size 17.78 8.89)
+		(margins 0.9525 0.9525 0.9525 0.9525)
+		(stroke
+			(width 0)
+			(type solid)
+		)
+		(fill
+			(type none)
+		)
+		(effects
+			(font
+				(size 1.27 1.27)
+			)
+			(justify left top)
 		)
 	)

Commit message: Digital section done
Parts:
- added J601: Conn_01x02_Pin, Connector_PinHeader_2.54mm:PinHeader_1x02_P2.54mm_Vertical, symbol Connector:Conn_01x02_Pin
Connections:
- net 12Vin: now also J601.1 (Pin_1)
- net GND: now also J601.2 (Pin_2)

Commit message: Complete except for recommended changes
Parts:
- added TP601, TP602, TP603: TestPoint, TestPoint:TestPoint_Pad_2.0x2.0mm, symbol Connector:TestPoint
Connections:
- net +3V3A: now also TP602.1
- net -3V3A: now also TP601.1
- net GND: now also TP603.1
Other:
- note added: "Solderable power connector"
- moved on the sheet: J601

Commit message: Temp probe bom done
Parts:
- added C613: 4.7uf, Capacitor_SMD:C_0603_1608Metric, symbol Device:C
- added C614, C615: 10uf, Capacitor_SMD:C_0603_1608Metric, symbol Device:C
- added D601: SMAJ24A, Diode_SMD:D_SMA, symbol Diode:SMAJ24A
- added R616: 500, Resistor_SMD:R_0603_1608Metric, symbol Device:R
- C601, C602, C606, C607, C609: MPN (none) -> GRM188R6YA106MA73D
- C603: MPN (none) -> C0603C105K4RACTU
- C604, C605: MPN (none) -> CL10B103KB8NNNC
- C608, C610, C611, C612: MPN (none) -> CL10A475KO8NNNC
- J601: now left out of the parts list
- P601: MPN (none) -> 436500200
- R601, R604: value 570k -> 569k; MPN (none) -> RN73H1JTTD5693B50
- R602, R603: MPN (none) -> ERA-3AEB184V
- R605, R608: MPN (none) -> ERA-3AEB3322V
- R606: value 499 -> 500; MPN (none) -> ERA-3AEB4990V
- R607, R609: value 200k -> 180k; MPN (none) -> ERA-3AEB184V
- R610: MPN (none) -> ERA-3AEB752V
- R611: value 453k -> 448k; MPN (none) -> RT0603BRD07448KL
- R612: value 49.9k -> 50k; MPN (none) -> RT0603BRD0750KL
- R613: value 450k -> 448k; MPN (none) -> RT0603BRD07448KL
- R614: MPN (none) -> RT0603BRD0750KL
- U601: MPN (none) -> LTC3260EMSE#TRPBF
- U602: MPN (none) -> LT3094EMSE#TRPBF
- U603: MPN (none) -> LT3042EMSE#TRPBF
Connections:
- net -3V3A: now also C613.2
- net 12Vin: now also C615.1, R616.2; no longer J601.1 (Pin_1), P601.1
- net GND: now also C613.1, C614.2, C615.2, D601.2 (A2)
- new net vin: C614.1, D601.1 (A1), J601.1 (Pin_1), P601.1, R616.1
Other:
- moved on the sheet: P601, TP603
