File: Circuit Boards/Black_Body_Temperature_Sensor_PCB/uA_current.kicad_sch (KiCad schematic)
At the start: 12 parts, among them Q5 TMUX1112PWR, Q6 TMUX1112PWR, U1 LM334M

Commit message: power simulation
Changed lines of the file:
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@@
-		)
-	)
-	(label "\"sel_t\"{1mA 100uA 10uA 1uA}"
-		(at 215.9 119.38 0)
-		(effects
-			(font
-				(size 1.27 1.27)
-			)
-			(justify left bottom)
 		)
 	)
@@
 		(effects
 			(font
-				(size 1.27 1.27)
-			)
-			(justify left bottom)
-		)
-	)
-	(label "\"sel_v\"{1mA 100uA 10uA 1uA}"
-		(at 175.26 91.44 0)
-		(effects
-			(font

Commit message: Schematic ready for review
Connections:
- net 100uA_T: now also R4.2; no longer R3.2
- net 100uA_V: now also R3.2; no longer R3.1, R4.1
- net 10uA_T: now also R6.2; no longer R5.2
- net 10uA_V: now also R5.2; no longer R5.1, R6.1
- net 1mA_T: now also R2.2; no longer R1.2
- net 1mA_V: now also R1.2; no longer R1.1, R2.1
- net 1uA_T: now also R8.2; no longer R7.2
- net 1uA_V: now also R7.2; no longer R7.1, R8.1
- net LM334_R: now also R1.1, R2.1, R3.1, R4.1, R5.1, R6.1, R7.1, R8.1
- net uA_I_Source: no longer R2.2, R4.2, R6.2, R8.2
- net +4V renamed +3V3A
Changed lines of the file:
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@@
 	(bus
 		(pts
-			(xy 172.72 91.44) (xy 205.74 91.44)
+			(xy 172.72 88.9) (xy 176.53 88.9)
 		)
 		(stroke
@@
 	(wire
 		(pts
-			(xy 234.95 50.8) (xy 224.79 50.8)
+			(xy 234.95 50.8) (xy 214.63 50.8)
 		)
 		(stroke
@@
 	(wire
 		(pts
-			(xy 133.35 49.53) (xy 133.35 48.26)
+			(xy 133.35 50.8) (xy 133.35 48.26)
 		)
 		(stroke
@@
 	(bus
 		(pts
-			(xy 214.63 120.65) (xy 214.63 119.38)
+			(xy 214.63 120.65) (xy 214.63 118.11)
 		)
 		(stroke
@@
 	(bus
 		(pts
-			(xy 214.63 119.38) (xy 246.38 119.38)
+			(xy 214.63 118.11) (xy 217.17 118.11)
 		)
 		(stroke
@@
 	(wire
 		(pts
-			(xy 173.99 50.8) (xy 184.15 50.8)
+			(xy 163.83 50.8) (xy 184.15 50.8)
 		)
 		(stroke
@@
 	(bus
 		(pts
-			(xy 172.72 91.44) (xy 172.72 99.06)
+			(xy 172.72 88.9) (xy 172.72 99.06)
 		)
 		(stroke
@@
 	(wire
 		(pts
-			(xy 123.19 49.53) (xy 133.35 49.53)
+			(xy 113.03 50.8) (xy 133.35 50.8)
 		)
 		(stroke
@@
 	(wire
 		(pts
-			(xy 71.12 50.8) (xy 82.55 50.8)
+			(xy 62.23 50.8) (xy 82.55 50.8)
 		)
 		(stroke
@@
 			(width 0)
 			(type default)
+		)
+	)
+	(label "100uA_T"
+		(at 113.03 50.8 0)
+		(effects
+			(font
+				(size 1.27 1.27)
+			)
+			(justify left bottom)
 		)
 	)
@@
 		)
 	)
+	(label "1mA_T"
+		(at 62.23 50.8 0)
+		(effects
+			(font
+				(size 1.27 1.27)
+			)
+			(justify left bottom)
+		)
+	)
 	(label "sel_v.100uA"
 		(at 154.94 96.52 0)
@@
 		)
 	)
-	(label "1uA_V"
+	(label "LM334_R"
+		(at 163.83 31.75 0)
+		(effects
+			(font
+				(size 1.27 1.27)
+			)
+			(justify left bottom)
+		)
+	)
+	(label "LM334_R"
+		(at 62.23 31.75 0)
+		(effects
+			(font
+				(size 1.27 1.27)
+			)
+			(justify left bottom)
+		)
+	)
+	(label "LM334_R"
+		(at 113.03 31.75 0)
+		(effects
+			(font
+				(size 1.27 1.27)
+			)
+			(justify left bottom)
+		)
+	)
+	(label "LM334_R"
 		(at 214.63 31.75 0)
 		(effects
@@
 		)
 	)
-	(label "10uA_T"
-		(at 163.83 43.18 0)
+	(label "1uA_T"
+		(at 214.63 50.8 0)
 		(effects
 			(font
@@
 	)
 	(label "1uA_T"
-		(at 214.63 43.18 0)
-		(effects
-			(font
-				(size 1.27 1.27)
-			)
-			(justify left bottom)
-		)
-	)
-	(label "1uA_T"
 		(at 210.82 118.11 180)
 		(effects
@@
 		)
 	)
-	(label "100uA_T"
+	(label "100uA_V"
 		(at 113.03 43.18 0)
+		(effects
+			(font
+				(size 1.27 1.27)
+			)
+			(justify left bottom)
+		)
+	)
+	(label "10uA_T"
+		(at 163.83 50.8 0)
 		(effects
 			(font
@@
 		)
 	)
-	(label "100uA_V"
-		(at 113.03 31.75 0)
-		(effects
-			(font
-				(size 1.27 1.27)
-			)
-			(justify left bottom)
-		)
-	)
 	(label "LM334M_V-"
 		(at 105.41 106.68 0)
@@
 		)
 	)
+	(label "1mA_V"
+		(at 62.23 43.18 0)
+		(effects
+			(font
+				(size 1.27 1.27)
+			)
+			(justify left bottom)
+		)
+	)
 	(label "10uA_V"
-		(at 163.83 31.75 0)
+		(at 163.83 43.18 0)
 		(effects
 			(font
@@
 		)
 	)
-	(label "1mA_V"
-		(at 62.23 31.75 0)
-		(effects
-			(font
-				(size 1.27 1.27)
-			)
-			(justify left bottom)
-		)
-	)
-	(label "1mA_T"
-		(at 62.23 43.18 0)
+	(label "1uA_V"
+		(at 214.63 43.18 0)
 		(effects
 			(font
@@
 			)
 			(justify right bottom)
-		)
-	)
-	(hierarchical_label "uA_I_Source"
-		(shape input)
-		(at 224.79 50.8 180)
-		(effects
-			(font
-				(size 1.27 1.27)
-			)
-			(justify right)
 		)
 	)
@@
 	(hierarchical_label "\"sel_v\"{1mA 100uA 10uA 1uA}"
 		(shape input)
-		(at 205.74 91.44 0)
+		(at 176.53 88.9 0)
 		(effects
 			(font
@@
 	(hierarchical_label "\"sel_t\"{1mA 100uA 10uA 1uA}"
 		(shape input)
-		(at 246.38 119.38 0)
+		(at 217.17 118.11 0)
 		(effects
 			(font
@@
 			)
 			(justify left)
-		)
-	)
-	(hierarchical_label "uA_I_Source"
-		(shape input)
-		(at 71.12 50.8 180)
-		(effects
-			(font
-				(size 1.27 1.27)
-			)
-			(justify right)
-		)
-	)
-	(hierarchical_label "uA_I_Source"
-		(shape input)
-		(at 173.99 50.8 180)
-		(effects
-			(font
-				(size 1.27 1.27)
-			)
-			(justify right)
-		)
-	)
-	(hierarchical_label "uA_I_Source"
-		(shape input)
-		(at 123.19 49.53 180)
-		(effects
-			(font
-				(size 1.27 1.27)
-			)
-			(justify right)
 		)
 	)
@@
 			)
 		)
-		(property "Value" "+4V"
+		(property "Value" "+3V3A"
 			(at 101.6 86.36 0)
 			(show_name no)

Commit message: Temp sensor schematic done
Parts:
- R201: renamed from R1; footprint (none) -> Resistor_SMD:R_0603_1608Metric
- R202: renamed from R2; footprint (none) -> Resistor_SMD:R_0603_1608Metric
- R203: renamed from R3; footprint (none) -> Resistor_SMD:R_0603_1608Metric
- R204: renamed from R4; footprint (none) -> Resistor_SMD:R_0603_1608Metric
- R205: renamed from R5; footprint (none) -> Resistor_SMD:R_0603_1608Metric
- R206: renamed from R6; footprint (none) -> Resistor_SMD:R_0603_1608Metric
- R207: renamed from R7; footprint (none) -> Resistor_SMD:R_0603_1608Metric
- R208: renamed from R8; footprint (none) -> Resistor_SMD:R_0603_1608Metric
- renumbered D5 to D201, Q5 to Q201, Q6 to Q202, U1 to U201
Other:
- note added: "uA Current (PAGE 2)"
- moved on the sheet: D201, Q201, Q202, R201, R202, R203, R204, R205, R206, R207, R208, U201

Commit message: temp pcb analog layout done
Connections:
- net 100uA_T: now also Q202.10 (D3); no longer Q202.15 (D2)
- net 100uA_V: now also Q201.7 (D4); no longer Q201.15 (D2)
- net 10uA_T: now also Q202.15 (D2); no longer Q202.10 (D3)
- net 10uA_V: now also Q201.2 (D1); no longer Q201.10 (D3)
- net 1mA_T: now also Q202.7 (D4); no longer Q202.2 (D1)
- net 1mA_V: now also Q201.10 (D3); no longer Q201.2 (D1)
- net 1uA_T: now also Q202.2 (D1); no longer Q202.7 (D4)
- net 1uA_V: now also Q201.15 (D2); no longer Q201.7 (D4)
- net sel_t.100uA: now also Q202.9 (SEL3); no longer Q202.16 (SEL2)
- net sel_t.10uA: now also Q202.16 (SEL2); no longer Q202.9 (SEL3)
- net sel_t.1mA: now also Q202.8 (SEL4); no longer Q202.1 (SEL1)
- net sel_t.1uA: now also Q202.1 (SEL1); no longer Q202.8 (SEL4)
- net sel_v.100uA: now also Q201.8 (SEL4); no longer Q201.16 (SEL2)
- net sel_v.10uA: now also Q201.1 (SEL1); no longer Q201.9 (SEL3)
- net sel_v.1mA: now also Q201.9 (SEL3); no longer Q201.1 (SEL1)
- net sel_v.1uA: now also Q201.16 (SEL2); no longer Q201.8 (SEL4)

Commit message: Complete except for recommended changes
Parts:
- added C201, C202, C203, C204, C205, C206, C207, C208, C209, C210, C211, C212, C213, C214, C215, C216: 2u2, Capacitor_SMD:C_0402_1005Metric, symbol Device:C
- added R201, R202, R203, R204, R205, R206, R207, R208: 5.1k, Resistor_SMD:R_0402_1005Metric, symbol Device:R
- D201: value 1N357 -> 1N457
- renumbered R201 to R209, R202 to R210, R203 to R211, R204 to R212, R205 to R213, R206 to R214, R207 to R215, R208 to R216
Connections:
- net GNDPWR: now also C201.2, C202.2, C203.2, C204.2, C205.2, C206.2, C207.2, C208.2, C209.2, C210.2, C211.2, C212.2, C213.2, C214.2, C215.2, C216.2
- net sel_t.100uA: now also C215.1, R207.2; no longer Q202.9 (SEL3)
- net sel_t.10uA: now also C214.1, R206.2; no longer Q202.16 (SEL2)
- net sel_t.1mA: now also C216.1, R208.2; no longer Q202.8 (SEL4)
- net sel_t.1uA: now also C213.1, R205.2; no longer Q202.1 (SEL1)
- net sel_v.100uA: now also C212.1, R204.2; no longer Q201.8 (SEL4)
- net sel_v.10uA: now also C209.1, R201.2; no longer Q201.1 (SEL1)
- net sel_v.1mA: now also C211.1, R203.2; no longer Q201.9 (SEL3)
- net sel_v.1uA: now also C210.1, R202.2; no longer Q201.16 (SEL2)
- new net selt1: C205.1, Q202.1 (SEL1), R205.1
- new net selt2: C206.1, Q202.16 (SEL2), R206.1
- new net selt3: C207.1, Q202.9 (SEL3), R207.1
- new net selt4: C208.1, Q202.8 (SEL4), R208.1
- new net selv1: C201.1, Q201.1 (SEL1), R201.1
- new net selv2: C202.1, Q201.16 (SEL2), R202.1
- new net selv3: C203.1, Q201.9 (SEL3), R203.1
- new net selv4: C204.1, Q201.8 (SEL4), R204.1
Other:
- moved on the sheet: D201, Q201, Q202, R209, R210, R211, R212, R213, R214, R215, R216, U201

Commit message: Temp probe bom done
Parts:
- C201, C202, C203, C204, C205, C206, C207, C208, C209, C210, C211, C212, C213, C214, C215, C216: MPN (none) -> GRM155R61E225ME15D
- D201: MPN (none) -> 1N457
- Q201, Q202: MPN (none) -> TMUX1112PWR
- R201, R202, R203, R204, R205, R206, R207, R208: MPN (none) -> RT0402BRD075K1L
- R209: value 134 -> 133; MPN (none) -> RQ73C1J133RBTD
- R210, R211: value 1.34k -> 1.33k; MPN (none) -> ERA-3AEB1331V
- R212, R213: value 13.4k -> 13.3k; MPN (none) -> ERA-3AEB1332V
- R214, R215: MPN (none) -> ERA-3AEB1333V
- R216: value 1.34M -> 1.33M; MPN (none) -> RK73H1JTTD1334F
- U201: MPN (none) -> LM334M
