File: Circuit Boards/Black_Body_Temperature_Sensor_PCB/micrcontroller.kicad_sch (KiCad schematic)
At the start: 32 parts, among them J701 Conn_01x06_Pin, J702 5040500891, J703 USB_C_Receptacle_USB2.0_16P, J704 Conn_01x04_Pin, P701 pogo programmer, SW701 SW_MEC_5E, SW702 SW_MEC_5E, U701 TXU0304, U702 ABM8G-25.000MHZ-18-D2Y-T, U703 USBLC6-2SC6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

Commit message: Designs finished - order placed
Parts:
- added D702: RED, LED_SMD:LED_0603_1608Metric, symbol Device:LED
- added R705: 1.33k, Resistor_SMD:R_0603_1608Metric, symbol Device:R
- U701: MPN TXU0304 -> TXU0304PWR
Connections:
- net +3V3: now also R705.2
- net GNDPWR: now also D702.1 (K)
- new net: D702.2 (A), R705.1
Other:
- note added: "POWER INDICATOR"
