File: Circuit Boards/Black_Body_Temperature_Sensor_PCB/Black_Body_Temperature_Sensor_PCB.kicad_pcb (KiCad board)
At the start: 6 copper layers, 62 x 77 mm, 217 parts, among them J401 Screw_Terminal_01x02, J402 Screw_Terminal_01x02, J601 Conn_01x02_Pin, J701 Conn_01x06_Pin, J702 5040500891, J703 USB_C_Receptacle_USB2.0_16P, J704 Conn_01x04_Pin, P601 436500200, P701 pogo programmer, Q201 TMUX1112PWR, Q202 TMUX1112PWR, Q301 TMUX1112PWR, Q401 TMUX1112PWR, Q402 TMUX1112PWR, Q403 TMUX1112PWR, SW701 SW_MEC_5E, SW702 SW_MEC_5E, U201 LM334M, U301 LM334M, U302 LT1008, U501 OPA376xxDBV, U502 OPA376xxDBV, U503 OPA376xxDBV, U504 OPA376xxDBV, U505 AD8421ARZ, U506 AD8421ARZ, U507 ADS131M04xPW, U508 ISO7762FDBQ, U509 OPA376xxDBV, U601 LTC3260xMSE, U602 LT3094xMSE, U603 LT3042xMSE, U701 TXU0304, U702 ABM8G-25.000MHZ-18-D2Y-T, U703 USBLC6-2SC6, U704 STM32G431RBTx, U705 AMS1117-3.3

Commit message: Minor rev.1 pcb changes. Firmware progress
Routing:
- net GND: vias 355 -> 353
- net (no net): vias 2 -> 4
