File: Circuit Boards/Black_Body_Heater_Control_PCB/ESP32.kicad_sch (KiCad schematic)
At the start: 24 parts, among them J201 5040500891, J202 Conn_01x04_Pin, J203 USB_C_Receptacle_USB2.0_16P, SW201 SW_MEC_5E, SW202 SW_MEC_5E, U201 AMS1117-3.3, U202 ESP32-S3-WROOM-1-N8R8, U203 USBLC6-2SC6

Commit message: Designs finished - order placed
Parts:
- C201: MPN (none) -> GRM188R6YA106MA73D
- C202, C204, C207: MPN (none) -> CL10B104KB8NNNC
- C203, C206: MPN (none) -> CL10A226MP8NUNE
- C205: MPN (none) -> C0603C105K4RACTU
- D201: MPN (none) -> LTST-C191KRKT
- R201, R203, R204, R205: MPN (none) -> ERA-3AEB103V
- R202: value 1k -> 1.33k; MPN (none) -> ERA-3AEB1331V
- R206, R207: footprint Resistor_SMD:R_0603_1608Metric -> Resistor_SMD:R_0402_1005Metric; MPN (none) -> RT0402BRD075K1L
Changed lines of the file:
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@@
 			)
 		)
+		(property "MPN" "CL10A226MP8NUNE"
+			(at 59.69 110.49 0)
+			(hide yes)
+			(show_name no)
+			(do_not_autoplace no)
+			(effects
+				(font
+					(size 1.27 1.27)
+				)
+			)
+		)
 		(pin "2"
 		)
@@
 			)
 		)
+		(property "MPN" "CL10B104KB8NNNC"
+			(at 91.44 62.23 0)
+			(hide yes)
+			(show_name no)
+			(do_not_autoplace no)
+			(effects
+				(font
+					(size 1.27 1.27)
+				)
+			)
+		)
 		(pin "2"
 		)
@@
 			)
 		)
+		(property "MPN" "CL10B104KB8NNNC"
+			(at 149.86 57.15 0)
+			(hide yes)
+			(show_name no)
+			(do_not_autoplace no)
+			(effects
+				(font
+					(size 1.27 1.27)
+				)
+			)
+		)
 		(pin "2"
 		)
@@
 			)
 		)
+		(property "MPN" "ERA-3AEB103V"
+			(at 53.34 54.61 0)
+			(hide yes)
+			(show_name no)
+			(do_not_autoplace no)
+			(effects
+				(font
+					(size 1.27 1.27)
+				)
+			)
+		)
 		(pin "2"
 		)
@@
 			)
 		)
-		(property "Footprint" "Resistor_SMD:R_0603_1608Metric"
+		(property "Footprint" "Resistor_SMD:R_0402_1005Metric"
 			(at 219.71 60.452 90)
 			(hide yes)
@@
 			)
 		)
+		(property "MPN" "RT0402BRD075K1L"
+			(at 219.71 62.23 90)
+			(hide yes)
+			(show_name no)
+			(do_not_autoplace no)
+			(effects
+				(font
+					(size 1.27 1.27)
+				)
+			)
+		)
 		(pin "2"
 		)
@@
 			)
 		)
-		(property "Footprint" "Resistor_SMD:R_0603_1608Metric"
+		(property "Footprint" "Resistor_SMD:R_0402_1005Metric"
 			(at 219.71 62.992 90)
 			(hide yes)
@@
 			)
 		)
+		(property "MPN" "RT0402BRD075K1L"
+			(at 219.71 64.77 90)
+			(hide yes)
+			(show_name no)
+			(do_not_autoplace no)
+			(effects
+				(font
+					(size 1.27 1.27)
+				)
+			)
+		)
 		(pin "2"
 		)
@@
 			)
 		)
+		(property "MPN" "ERA-3AEB103V"
+			(at 186.69 115.57 90)
+			(hide yes)
+			(show_name no)
+			(do_not_autoplace no)
+			(effects
+				(font
+					(size 1.27 1.27)
+				)
+			)
+		)
 		(pin "2"
 		)
@@
 			)
 		)
+		(property "MPN" "CL10B104KB8NNNC"
+			(at 50.8 62.23 0)
+			(hide yes)
+			(show_name no)
+			(do_not_autoplace no)
+			(effects
+				(font
+					(size 1.27 1.27)
+				)
+			)
+		)
 		(pin "2"
 		)
@@
 			)
 		)
+		(property "MPN" "GRM188R6YA106MA73D"
+			(at 31.75 110.49 0)
+			(hide yes)
+			(show_name no)
+			(do_not_autoplace no)
+			(effects
+				(font
+					(size 1.27 1.27)
+				)
+			)
+		)
 		(pin "1"
 		)
@@
 			)
 		)
+		(property "MPN" "CL10A226MP8NUNE"
+			(at 137.16 57.15 0)
+			(hide yes)
+			(show_name no)
+			(do_not_autoplace no)
+			(effects
+				(font
+					(size 1.27 1.27)
+				)
+			)
+		)
 		(pin "2"
 		)
@@
 			)
 		)
-		(property "Value" "1k"
+		(property "Value" "1.33k"
 			(at 88.9 113.0299 0)
 			(show_name no)
@@
 			)
 		)
+		(property "MPN" "ERA-3AEB1331V"
+			(at 86.36 111.76 0)
+			(hide yes)
+			(show_name no)
+			(do_not_autoplace no)
+			(effects
+				(font
+					(size 1.27 1.27)
+				)
+			)
+		)
 		(pin "2"
 		)
@@
 			)
 		)
+		(property "MPN" "LTST-C191KRKT"
+			(at 86.36 120.65 90)
+			(hide yes)
+			(show_name no)
+			(do_not_autoplace no)
+			(effects
+				(font
+					(size 1.27 1.27)
+				)
+			)
+		)
 		(pin "1"
 		)
@@
 			)
 		)
+		(property "MPN" "ERA-3AEB103V"
+			(at 128.27 110.49 90)
+			(hide yes)
+			(show_name no)
+			(do_not_autoplace no)
+			(effects
+				(font
+					(size 1.27 1.27)
+				)
+			)
+		)
 		(pin "2"
 		)
@@
 			)
 		)
+		(property "MPN" "ERA-3AEB103V"
+			(at 93.98 54.61 0)
+			(hide yes)
+			(show_name no)
+			(do_not_autoplace no)
+			(effects
+				(font
+					(size 1.27 1.27)
+				)
+			)
+		)
 		(pin "2"
 		)
@@
 			(at 134.62 115.57 0)
 			(hide yes)
+			(show_name no)
+			(do_not_autoplace no)
+			(effects
+				(font
+					(size 1.27 1.27)
+				)
+			)
+		)
+		(property "MPN" "C0603C105K4RACTU"
+			(at 134.62 115.57 0)
+			(hide yes)
